Commit message: Position control topic implemented.

File: stereo_bot_description/urdf/stereo_bot.xacro (robot description, xacro)
@@ -125,13 +125,13 @@
 	<child link="neck"/>
 	<axis xyz="0 0 1"/>
-	<limit lower="-1.5707963" upper="1.5707963" effort="10" velocity="30"/>
+	<limit lower="-1.5707963" upper="1.5707963" effort="1000" velocity="1"/>
 </joint>
 <transmission name="transmission">
 	<type>transmission_interface/SimpleTransmission</type>
 	<joint name="neck_to_base">
-		<hardwareInterface>EffortJointInterface</hardwareInterface>
+		<hardwareInterface>PositionJointInterface</hardwareInterface>
 	</joint>
 	<actuator name="neck_actuator">
-		<hardwareInterface>EffortJointInterface</hardwareInterface>
+		<hardwareInterface>PositionJointInterface</hardwareInterface>
 		<mechanicalReduction>1</mechanicalReduction>
 	</actuator>
